File: GepRev2.kicad_sch (KiCad schematic)
At the start: 79 parts

Commit message: more work on shematic
Parts:
- removed D? (x4): DIODE, symbol Simulation_SPICE:DIODE
- removed MX? (x4): MX-NoLED, symbol MX_Alps_Hybrid:MX-NoLED
- added D? (x65): DIODE, symbol Simulation_SPICE:DIODE
- added J?: Conn_02x10_Top_Bottom, symbol Connector_Generic:Conn_02x10_Top_Bottom
- added MX? (x55): MX-NoLED, symbol MX_Alps_Hybrid:MX-NoLED
- added U?: RSTSWITCH, symbol keebio:PRTR5V0U2X
- added U?: BRKOUT, symbol keebio:PRTR5V0U2X
Connections:
- net COL0 is gone; now on net PIN0: MX?.1 (COL), MX?.1 (COL), MX?.1 (COL), MX?.1 (COL)
- net COL1 is gone; now on net PIN1: MX?.1 (COL), MX?.1 (COL), MX?.1 (COL), MX?.1 (COL)
- net COL2 is gone; now on net PIN2: MX?.1 (COL), MX?.1 (COL), MX?.1 (COL), MX?.1 (COL)
- net COL3 is gone; now on net PIN3: MX?.1 (COL), MX?.1 (COL), MX?.1 (COL), MX?.1 (COL)
- net COL4 is gone; now on net PIN4: MX?.1 (COL), MX?.1 (COL), MX?.1 (COL), MX?.1 (COL)
- net COL5 is gone; now on net PIN5: MX?.1 (COL), MX?.1 (COL), MX?.1 (COL), MX?.1 (COL), MX?.1 (COL)
- net COL6 is gone; now on net PIN6: MX?.1 (COL), MX?.1 (COL), MX?.1 (COL), MX?.1 (COL), MX?.1 (COL)
- net COL7 is gone; now on net PIN7: MX?.1 (COL), MX?.1 (COL), MX?.1 (COL), MX?.1 (COL), MX?.1 (COL)
- net PIN9: now reaches U?.11 (P1.04)
- net PIN9: now also D?.2 (K), MX?.1 (COL), MX?.1 (COL), MX?.1 (COL), MX?.1 (COL), MX?.1 (COL), MX?.1 (COL), MX?.1 (COL), MX?.1 (COL), MX?.1 (COL)
- net PIN8: now reaches U?.12 (P1.06)
- net PIN8: now also D?.2 (K), MX?.1 (COL), MX?.1 (COL), MX?.1 (COL), MX?.1 (COL), MX?.1 (COL), MX?.1 (COL), MX?.1 (COL), MX?.1 (COL), MX?.1 (COL)
- net PIN7: now reaches U?.13 (NFC1/P0.09)
- net PIN7: now also D?.2 (K), MX?.1 (COL), MX?.1 (COL), MX?.1 (COL), MX?.1 (COL)
- net PIN6: now reaches U?.14 (NFC2/P0.10)
- net PIN6: now also D?.2 (K), MX?.1 (COL), MX?.1 (COL), MX?.1 (COL), MX?.1 (COL)
- net PIN5: now reaches U?.15 (P1.11)
- net PIN5: now also D?.2 (K), MX?.1 (COL), MX?.1 (COL), MX?.1 (COL), MX?.1 (COL)
- net PIN4: now reaches U?.16 (P1.13)
- net PIN4: now also D?.2 (K), MX?.1 (COL), MX?.1 (COL), MX?.1 (COL), MX?.1 (COL), MX?.1 (COL)
- net PIN3: now reaches U?.17 (P1.15)
- net PIN3: now also D?.2 (K), MX?.1 (COL), MX?.1 (COL), MX?.1 (COL), MX?.1 (COL), MX?.1 (COL)
- net PIN2: now reaches U?.18 (AIN0/P0.02)
- net PIN2: now also D?.2 (K), MX?.1 (COL), MX?.1 (COL), MX?.1 (COL), MX?.1 (COL), MX?.1 (COL)
- net PIN1: now reaches U?.19 (AIN5/P0.29)
- net PIN1: now also D?.2 (K), MX?.1 (COL), MX?.1 (COL), MX?.1 (COL), MX?.1 (COL), MX?.1 (COL)
- net PIN0: now reaches U?.20 (AIN7/P0.31)
- net PIN0: now also D?.2 (K), MX?.1 (COL), MX?.1 (COL), MX?.1 (COL), MX?.1 (COL), MX?.1 (COL)
- net +5V: now reaches U?.21 (VCC)
- net +5V: now also U?.2 (I/O1)
- net RST: now reaches U?.22 (RST)
- net RST: now also U?.1 (GND)
- net GND: now reaches U?.23 (GND)
- net GND: now also U?.3 (GND), U?.4 (GND), U?.1 (GND), U?.2 (I/O1)
- net SDA: now reaches U?.5 (P0.17)
- net SDA: now also U?.4 (VCC)
- net SCL: now reaches U?.6 (P0.20)
- net SCL: now also U?.3 (I/O2)
- net ROW0: no longer names the net of D?.2 (K), D?.2 (K), D?.2 (K), D?.2 (K), D?.2 (K), D?.2 (K), D?.2 (K)
- net ROW0: now also D?.1 (A), D?.2 (K), D?.2 (K)
- net ROW1: no longer names the net of D?.2 (K), D?.2 (K), D?.2 (K), D?.2 (K), D?.2 (K), D?.2 (K), D?.2 (K)
- net ROW1: now also D?.1 (A), D?.2 (K), D?.2 (K)
- net ROW2: no longer names the net of D?.2 (K), D?.2 (K), D?.2 (K), D?.2 (K), D?.2 (K), D?.2 (K), D?.2 (K)
- net ROW2: now also D?.1 (A), D?.2 (K), D?.2 (K)
- net ROW3: no longer names the net of D?.2 (K), D?.2 (K), D?.2 (K), D?.2 (K), D?.2 (K), D?.2 (K), D?.2 (K)
- net ROW3: now also D?.1 (A), D?.2 (K), D?.2 (K)
- net ROW4: no longer names the net of D?.2 (K), D?.2 (K), D?.2 (K), D?.2 (K), D?.2 (K), D?.2 (K), D?.2 (K)
- net ROW4: now also D?.1 (A), D?.2 (K), D?.2 (K)
- new net: D?.1 (A), MX?.2 (ROW) (x55)
- new net: D?.1 (A), D?.2 (K), D?.2 (K), D?.2 (K), D?.2 (K), D?.2 (K), D?.2 (K), D?.2 (K), D?.2 (K), D?.2 (K) (x5)
Other:
- moved on the sheet: D?, MX?, U?

Commit message: Updates to schematic
Parts:
- added J?: Conn_02x10_Top_Bottom_Left, symbol Connector_Generic:Conn_02x10_Top_Bottom
- added R? (x6): R_Small, symbol Device:R_Small
- added SW? (x2): RotaryEncoder, symbol Device:RotaryEncoder
- J?: value Conn_02x10_Top_Bottom -> Conn_02x10_Top_Bottom_Right
Connections:
- net +5V: now also R?.1, R?.1, R?.1, R?.2, R?.2, R?.2
- net GND: now also SW?.C, SW?.C
- net PIN0: now also J?.1 (Pin_1); no longer MX?.1 (COL), MX?.1 (COL), MX?.1 (COL), MX?.1 (COL), MX?.1 (COL)
- net PIN1: now also J?.2 (Pin_2); no longer MX?.1 (COL), MX?.1 (COL), MX?.1 (COL), MX?.1 (COL), MX?.1 (COL)
- net PIN2: now also J?.3 (Pin_3); no longer MX?.1 (COL), MX?.1 (COL), MX?.1 (COL), MX?.1 (COL), MX?.1 (COL)
- net PIN3: now also J?.4 (Pin_4); no longer MX?.1 (COL), MX?.1 (COL), MX?.1 (COL), MX?.1 (COL), MX?.1 (COL)
- net PIN4: now also J?.5 (Pin_5); no longer MX?.1 (COL), MX?.1 (COL), MX?.1 (COL), MX?.1 (COL), MX?.1 (COL)
- net PIN5: now also J?.6 (Pin_6); no longer D?.2 (K), MX?.1 (COL), MX?.1 (COL), MX?.1 (COL), MX?.1 (COL)
- net PIN6: now also J?.7 (Pin_7); no longer D?.2 (K), MX?.1 (COL), MX?.1 (COL), MX?.1 (COL), MX?.1 (COL)
- net PIN7: now also J?.8 (Pin_8); no longer D?.2 (K), MX?.1 (COL), MX?.1 (COL), MX?.1 (COL), MX?.1 (COL)
- net PIN8: now also J?.9 (Pin_9); no longer D?.2 (K), MX?.1 (COL), MX?.1 (COL), MX?.1 (COL), MX?.1 (COL)
- net PIN9: now also J?.10 (Pin_10); no longer D?.2 (K), MX?.1 (COL), MX?.1 (COL), MX?.1 (COL), MX?.1 (COL)
- net SCL: now also R?.1
- net SDA: now also R?.2
- net REB_L: now reaches U?.10 (P0.11)
- net REB_L: now also J?.19 (Pin_19)
- net REA_R: now reaches U?.7 (P0.22)
- net REA_R: now also R?.2, SW?.A
- net REB_R: now reaches U?.8 (P0.24)
- net REB_R: now also R?.1, SW?.B
- net REA_L: now reaches U?.9 (P1.00)
- net REA_L: now also J?.20 (Pin_20)
- net PIN9_R: now reaches J?.1 (Pin_1)
- net PIN9_R: now also D?.2 (K), MX?.1 (COL), MX?.1 (COL), MX?.1 (COL), MX?.1 (COL)
- net PIN0_R: now reaches J?.10 (Pin_10)
- net PIN0_R: now also MX?.1 (COL), MX?.1 (COL), MX?.1 (COL), MX?.1 (COL), MX?.1 (COL)
- net PIN8_R: now reaches J?.2 (Pin_2)
- net PIN8_R: now also D?.2 (K), MX?.1 (COL), MX?.1 (COL), MX?.1 (COL), MX?.1 (COL)
- net PIN7_R: now reaches J?.3 (Pin_3)
- net PIN7_R: now also D?.2 (K), MX?.1 (COL), MX?.1 (COL), MX?.1 (COL), MX?.1 (COL)
- net PIN6_R: now reaches J?.4 (Pin_4)
- net PIN6_R: now also D?.2 (K), MX?.1 (COL), MX?.1 (COL), MX?.1 (COL), MX?.1 (COL)
- net PIN5_R: now reaches J?.5 (Pin_5)
- net PIN5_R: now also D?.2 (K), MX?.1 (COL), MX?.1 (COL), MX?.1 (COL), MX?.1 (COL)
- net PIN4_R: now reaches J?.6 (Pin_6)
- net PIN4_R: now also MX?.1 (COL), MX?.1 (COL), MX?.1 (COL), MX?.1 (COL), MX?.1 (COL)
- net PIN3_R: now reaches J?.7 (Pin_7)
- net PIN3_R: now also MX?.1 (COL), MX?.1 (COL), MX?.1 (COL), MX?.1 (COL), MX?.1 (COL)
- net PIN2_R: now reaches J?.8 (Pin_8)
- net PIN2_R: now also MX?.1 (COL), MX?.1 (COL), MX?.1 (COL), MX?.1 (COL), MX?.1 (COL)
- net PIN1_R: now reaches J?.9 (Pin_9)
- net PIN1_R: now also MX?.1 (COL), MX?.1 (COL), MX?.1 (COL), MX?.1 (COL), MX?.1 (COL)
- new net REA: J?.12 (Pin_12), R?.2, SW?.A
- new net REB: J?.11 (Pin_11), R?.1, SW?.B
Other:
- moved on the sheet: D?, J?, MX?, U?
